File: pcb/acro.kicad_pcb (KiCad board)
At the start: 2 copper layers, 36 x 36 mm, 27 parts, among them P1 CONN_01X02, Q1 Q_NMOS_GSD, U1 MPU-6500, U2 TLV70233DBV

Commit message: change pull up resistor value
Changed lines of the file:
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@@
     (effects (font (size 1 1) (thickness 0.15)))
   )
-  (gr_text ckd.tech/acro/v1 (at 145.09 117.58 360) (layer F.SilkS)
+  (gr_text ckd.tech/acro/v1 (at 145.09 117.58) (layer F.SilkS)
     (effects (font (size 1.25 1.25) (thickness 0.25)))
   )

Commit message: Add license information to many files. PCB design files are CC-BY and code is MIT license.
Other:
- board text added: "Copyright 2016 Chickadee Tech LLC, <add attributions here> This work is licensed under the Creative Commons Attribution 4.0 International License. To view a copy of this license, visit http://creativecommons.org/licenses/by/4.0/ or send a letter to Creative Commons, PO Box 1866, Mountain View, CA 94042, USA."
- board text added: "Remove all Chickadee Tech LLC trademarks before making your own board. The Chickadee logo and Polystack logo are owned by Chickadee Tech LLC. You may license the Polystack logo for free by emailing support@chickadee.tech and receiving express written permission from Chickadee Tech LLC."
Changed lines of the file:
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@@
-(kicad_pcb (version 4) (host pcbnew "(2015-11-03 BZR 6296)-product")
+(kicad_pcb (version 4) (host pcbnew 4.0.1-stable)
   (general
     (links 150)
@@
     (area 118.127143 74.1 205.267857 178)
     (thickness 1.6)
-    (drawings 37)
+    (drawings 40)
     (tracks 1014)
     (zones 0)
@@
     (40 Dwgs.User user)
     (41 Cmts.User user)
-    (42 Eco1.User user hide)
-    (43 Eco2.User user hide)
+    (42 Eco1.User user)
+    (43 Eco2.User user)
     (44 Edge.Cuts user)
     (45 Margin user)
@@
       (xy -2.200426 1.477507) (xy -2.158969 1.476897)) (layer B.Mask) (width 0.01))
   )
+  (gr_text "Copyright 2016 Chickadee Tech LLC, <add attributions here>\n\nThis work is licensed under the Creative Commons Attribution 4.0 International License.\nTo view a copy of this license, visit http://creativecommons.org/licenses/by/4.0/\nor send a letter to Creative Commons, PO Box 1866, Mountain View, CA 94042, USA." (at 178.85 173.61) (layer Cmts.User)
+    (effects (font (size 1.5 1.5) (thickness 0.3)) (justify left))
+  )
+  (gr_line (start 138.66 126.14) (end 116 129.99) (layer Cmts.User) (width 0.2))
+  (gr_text "Remove all Chickadee Tech LLC trademarks\nbefore making your own board. The\nChickadee logo and Polystack logo\nare owned by Chickadee Tech LLC.\n\nYou may license the Polystack logo for\nfree by emailing support@chickadee.tech\nand receiving express written permission\nfrom Chickadee Tech LLC." (at 92.12 140.71) (layer Cmts.User)
+    (effects (font (size 1.5 1.5) (thickness 0.3)) (justify left))
+  )
   (gr_text 50mA (at 164.91 107.96 90) (layer B.SilkS)
     (effects (font (size 1 1) (thickness 0.175)) (justify mirror))
@@
   (gr_line (start 166 92.75) (end 166 123.25) (angle 90) (layer Edge.Cuts) (width 0.15))
   (gr_line (start 132.75 90) (end 163.25 90) (angle 90) (layer Edge.Cuts) (width 0.15))
-  (gr_text acro (at 187.25 174.25) (layer Cmts.User)
-    (effects (font (size 5 5) (thickness 0.5)) (justify left))
+  (gr_text acro (at 186.34 189.49) (layer Cmts.User)
+    (effects (font (size 3 3) (thickness 0.5)) (justify left))
   )
   (segment (start 162.95 97.849974) (end 162.95 96.45) (width 0.1524) (layer F.Cu) (net 1))
